File: 2-bach.kicad_sch (KiCad schematic)
At the start: 0 parts

Commit message: Initial schematic entry
Lets get started
Other:
- added sheet PowerSupply (PowerSupply.kicad_sch)
Changed lines of the file:
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@@
+		)
+	)
+	(sheet
+		(at 87.63 68.072)
+		(size 50.038 26.67)
+		(exclude_from_sim no)
+		(in_bom yes)
+		(on_board yes)
+		(dnp no)
+		(fields_autoplaced yes)
+		(stroke
+			(width 0.1524)
+			(type solid)
+		)
+		(fill
+			(color 0 0 0 0)
+		)
+		(property "Sheetname" "PowerSupply"
+			(at 87.63 67.3604 0)
+			(show_name no)
+			(do_not_autoplace no)
+			(effects
+				(font
+					(size 1.27 1.27)
+				)
+				(justify left bottom)
+			)
+		)
+		(property "Sheetfile" "PowerSupply.kicad_sch"
+			(at 87.63 95.3266 0)
+			(show_name no)
+			(do_not_autoplace no)
+			(effects
+				(font
+					(size 1.27 1.27)
+				)
+				(justify left top)
+			)
+		)
+		(instances
+			(project "2-bach"
+				(path "/3db49100-90e5-41c8-b73a-56a81b787550"
+					(page "3")
+				)
+			)
 		)
 	)
