File: PowerStage.kicad_sch (KiCad schematic)
At the start: 28 parts, among them U1 ECC82/12AU7, U2 ECC81, U3 ECC82/12AU7

Commit message: minor updates
Other:
- title: (none) -> 2-Bach Amplifier
Changed lines of the file:
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@@
 	(generator_version "10.0")
 	(paper "A4")
+	(title_block
+		(title "2-Bach Amplifier")
+		(date "2026-07-26")
+		(rev "0.1")
+	)
 	(junction
 		(at 165.1 50.8)
