File: ReverbModule/Driver.kicad_sch (KiCad schematic)
At the start: 29 parts, among them J1 Tank, J2 Screw_Terminal_01x02, Q1 BD139, Q2 BD140, U1 NE5532

Commit message: starting layout
Connections:
- net TankIn+: now reaches C10.1, C9.2, D1.1 (K), D2.2 (A), J1.1 (In1), R7.2, R8.1, R9.1, U1.7
- net Q2B: now reaches C10.2, D2.1 (K), Q2.3 (B), R6.1
- net TankIn-: now reaches C8.1, J1.2 (Ext1), R4.1
- net Q1B: now reaches C9.1, D1.2 (A), Q1.3 (B), R5.2
Changed lines of the file:
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@@
 	(title_block
 		(title "Reverb Driver")
+		(date "2026-07-16")
+		(rev "0.1")
 	)
 	(text "Drive Level"
@@
 		)
 	)
+	(label "Q2B"
+		(at 200.66 76.2 0)
+		(effects
+			(font
+				(size 1.27 1.27)
+			)
+			(justify left bottom)
+		)
+	)
+	(label "Q1B"
+		(at 200.406 50.8 0)
+		(effects
+			(font
+				(size 1.27 1.27)
+			)
+			(justify left bottom)
+		)
+	)
+	(label "TankIn+"
+		(at 226.06 63.5 0)
+		(effects
+			(font
+				(size 1.27 1.27)
+			)
+			(justify left bottom)
+		)
+	)
+	(label "TankIn-"
+		(at 238.76 104.14 0)
+		(effects
+			(font
+				(size 1.27 1.27)
+			)
+			(justify left bottom)
+		)
+	)
