File: ReverbModule/Recovery.kicad_sch (KiCad schematic)
At the start: 0 parts

Commit message: In worl
Parts:
- added J1: Tank, symbol Connector:Conn_Coaxial_x2_Isolated
- added U2: NE5532, symbol Amplifier_Operational:NE5532

Commit message: More Schematic Capture
Parts:
- added C5, C6: 100nF, Capacitor_SMD:C_0805_2012Metric_Pad1.18x1.45mm_HandSolder, symbol Device:C
- added unit 3 of U2
Connections:
- new net: C5.1, U2.8 (V+)
- new net: C6.2, U2.4 (V-)
- new net GND: C5.2, C6.1

Commit message: in progress
Parts:
- added C13: 100nF, Capacitor_SMD:C_1210_3225Metric_Pad1.33x2.70mm_HandSolder, symbol Device:C
- added C14: 10nF, Capacitor_SMD:C_1206_3216Metric_Pad1.33x1.80mm_HandSolder, symbol Device:C
- added C15, C17, C18: 10µF, Capacitor_SMD:CP_Elec_5x5.3, symbol Device:C_Polarized_US
- added C16: 220p, Capacitor_SMD:C_0805_2012Metric_Pad1.18x1.45mm_HandSolder, symbol Device:C
- added R10: 4.7k, Resistor_SMD:R_0805_2012Metric_Pad1.20x1.40mm_HandSolder, symbol Device:R_US
- added R11: 100k, Resistor_SMD:R_0805_2012Metric_Pad1.20x1.40mm_HandSolder, symbol Device:R_US
- added R12: 560R, Resistor_SMD:R_0805_2012Metric_Pad1.20x1.40mm_HandSolder, symbol Device:R_US
- added R13, R15: R_US, symbol Device:R_US
- added R14: 22k, Resistor_SMD:R_0805_2012Metric_Pad1.20x1.40mm_HandSolder, symbol Device:R_US
Connections:
- net GND: now also J1.4 (Ext2), C15.2, R10.2, R11.2
- net at U2.5 (+): now also R12.2
- net at U2.6 (-): now also C16.1, R13.1, R14.1
- net at U2.7: now also C16.2, R14.2, R15.1
- net at J1.3 (In2): now also C13.2
- new net: C17.2, R15.2
- new net: C14.2, R10.1
- new net: C13.1, C14.1, R11.1, R12.1
- new net: C15.1, R13.2
Other:
- moved on the sheet: J1B, U2A, U2B

Commit message: Schematic Capture
Parts:
- added J3: Foot_Switch, TerminalBlock_Phoenix:TerminalBlock_Phoenix_MKDS-3-2-5.08_1x02_P5.08mm_Horizontal, symbol Connector:Screw_Terminal_01x02
- added J4: Screw_Terminal_01x02, TerminalBlock_Phoenix:TerminalBlock_Phoenix_MKDS-3-2-5.08_1x02_P5.08mm_Horizontal, symbol Connector:Screw_Terminal_01x02
- added J5: Screw_Terminal_01x03, symbol Connector:Screw_Terminal_01x03
- added R17: 22k, Resistor_SMD:R_0805_2012Metric_Pad1.20x1.40mm_HandSolder, symbol Device:R_US
- added R19: 10k, Resistor_SMD:R_0805_2012Metric_Pad1.20x1.40mm_HandSolder, symbol Device:R_US
- added RV3: 10K, symbol Device:R_Potentiometer_US
- R13: value R_US -> 220; footprint (none) -> Resistor_SMD:R_0805_2012Metric_Pad1.20x1.40mm_HandSolder; LCSC (none) -> C17557; MPN (none) -> 0805W8F2200T5E
- R15: value R_US -> 560; footprint (none) -> Resistor_SMD:R_0805_2012Metric_Pad1.20x1.40mm_HandSolder; LCSC (none) -> C28636
Connections:
- net GND: now also U2.3 (+), J3.2 (Pin_2), J4.2 (Pin_2), J5.2 (Pin_2), R17.1, RV3.3
- net at C17.1: now also J3.1 (Pin_1), RV3.1
- net at U2.1: now also C18.2, R19.2
- net Dry: now reaches U2.2 (-)
- net Dry: now also R19.1, RV3.2
- net +15V: now reaches C5.1, U2.8 (V+)
- net +15V: now also J5.1 (Pin_1)
- net -15V: now reaches C6.2, U2.4 (V-)
- net -15V: now also J5.3 (Pin_3)
- net at C18.1: now also J4.1 (Pin_1), R17.2
Other:
- note added: "Tank Output"
- moved on the sheet: C5

Commit message: Capture Complete
Parts:
- J1: footprint (none) -> TerminalBlock_Phoenix:TerminalBlock_Phoenix_MKDS-1,5-2-5.08_1x02_P5.08mm_Horizontal
- J5, RV3: footprint (none) -> TerminalBlock_Phoenix:TerminalBlock_Phoenix_MKDS-1,5-3-5.08_1x03_P5.08mm_Horizontal
- U2: footprint (none) -> Package_SO:SOIC-8_3.9x4.9mm_P1.27mm
Changed lines of the file:
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@@
 			)
 		)
-		(property "Footprint" ""
+		(property "Footprint" "Package_SO:SOIC-8_3.9x4.9mm_P1.27mm"
 			(at 185.42 78.74 0)
 			(hide yes)
@@
 			)
 		)
-		(property "Footprint" ""
+		(property "Footprint" "Package_SO:SOIC-8_3.9x4.9mm_P1.27mm"
 			(at 101.6 76.2 0)
 			(hide yes)
@@
 			)
 		)
-		(property "Footprint" ""
+		(property "Footprint" "TerminalBlock_Phoenix:TerminalBlock_Phoenix_MKDS-1,5-3-5.08_1x03_P5.08mm_Horizontal"
 			(at 162.56 82.55 0)
 			(hide yes)
@@
 			)
 		)
-		(property "Footprint" ""
+		(property "Footprint" "TerminalBlock_Phoenix:TerminalBlock_Phoenix_MKDS-1,5-3-5.08_1x03_P5.08mm_Horizontal"
 			(at 68.58 139.7 0)
 			(hide yes)
@@
 			)
 		)
-		(property "Footprint" ""
+		(property "Footprint" "TerminalBlock_Phoenix:TerminalBlock_Phoenix_MKDS-1,5-2-5.08_1x02_P5.08mm_Horizontal"
 			(at 43.18 81.28 0)
 			(hide yes)
@@
 			)
 		)
-		(property "Footprint" ""
+		(property "Footprint" "Package_SO:SOIC-8_3.9x4.9mm_P1.27mm"
 			(at 43.18 142.24 0)
 			(hide yes)
