File: ReverbModule/ReverbModule.kicad_pcb (KiCad board)
At the start: 2 copper layers, 50 parts, among them J1 Tank, J2 Screw_Terminal_01x02, J3 Foot_Switch, J4 Screw_Terminal_01x02, J5 Screw_Terminal_01x03, Q1 BD139, Q2 BD140, U1 NE5532, U2 NE5532

Commit message: ub wirj
Parts:
- added H1: M3, MountingHole:MountingHole_3.2mm_M3, F.Cu at (94.9, 85.0)
- added H2: M3, MountingHole:MountingHole_3.2mm_M3, F.Cu at (94.9, 45.0)
- added H3: M3, MountingHole:MountingHole_3.2mm_M3, F.Cu at (184.9, 85.0)
- added H4: M3, MountingHole:MountingHole_3.2mm_M3, F.Cu at (184.9, 45.0)
- added H5: M3, MountingHole:MountingHole_3.2mm_M3, F.Cu at (94.9, 95.0)
- added H6: M3, MountingHole:MountingHole_3.2mm_M3, F.Cu at (184.9, 95.0)
- added H7: M3, MountingHole:MountingHole_3.2mm_M3, F.Cu at (94.9, 135.1)
- added H8: M3, MountingHole:MountingHole_3.2mm_M3, F.Cu at (184.9, 135.1)
- added TP1: TestPoint, TestPoint:TestPoint_THTPad_D4.0mm_Drill2.0mm, F.Cu at (184.9, 115.0)
Routing:
- added copper zone on B.Cu, net GND
- added copper zone on F.Cu, net GND
Other:
- board outline added: 100 x 100 mm
- board text added: "MaxPlate 100x100 Andrew Fischer 21012022"
