File: ReverbModule/ReverbModule.kicad_pcb (KiCad board)
At the start: 2 copper layers, 100 x 100 mm, 59 parts, among them J1 Tank, J2 Screw_Terminal_01x02, J3 Foot_Switch, J4 Screw_Terminal_01x02, J5 Screw_Terminal_01x03, Q1 BD139, Q2 BD140, U1 NE5532, U2 NE5532

Commit message: starting layout
Parts:
- moved C1 59.2 mm to (163.0, 47.0)
- moved R2 58.9 mm to (172.0, 53.0)
- moved J3 57.7 mm to (158.7, 124.0)
- moved U1 54.0 mm to (150.0, 59.0)
- moved R1 52.4 mm to (166.0, 53.0)
- moved C2 51.4 mm to (138.0, 57.0)
- moved R18 40.8 mm to (138.0, 62.0), turned to 180 degrees
- moved D1 35.6 mm to (162.0, 58.0)
- moved C8 34.8 mm to (158.0, 67.5), turned to 90 degrees
- moved J2 25.6 mm to (147.5, 47.1)
- moved C7 25.4 mm to (132.0, 57.0), turned to 180 degrees
- moved RV1 23.7 mm to (127.9, 47.2)
- moved C16 21.4 mm to (184.0, 102.0)
- moved RV2 15.3 mm to (107.2, 65.1), turned to 90 degrees
- moved R4 14.7 mm to (144.0, 67.0)
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Connections:
- net Net-(D1-A) renamed /Driver/Q1B
- net Net-(D1-K) renamed /Driver/Q2B
- net Net-(J1A-Ext1) renamed /Driver/TankIn-
