File: Dual15PowerSupply/Dual15PowerSupply.kicad_sch (KiCad schematic)
At the start: 34 parts, among them J1 120VAC, J2 +/-15VDC, U1 LT3091, U2 LT3081

Commit message: DRC cleanups
Parts:
- D1: Mouser 241-RPMS210_R2_00601 -> 241-RPMS210_R2_00601
Changed lines of the file:
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@@
 		(in_pos_files yes)
 		(dnp no)
-		(fields_autoplaced yes)
 		(property "Reference" "D1"
-			(at 100.33 40.7668 90)
+			(at 102.87 40.7668 90)
 			(show_name no)
 			(do_not_autoplace no)
@@
 		)
 		(property "Value" "RPMS210"
-			(at 100.33 43.3068 90)
+			(at 102.87 43.307 90)
 			(show_name no)
 			(do_not_autoplace no)
@@
 			)
 		)
-		(property "Mouser" "241-RPMS210_R2_00601 "
+		(property "Mouser" "241-RPMS210_R2_00601"
 			(at 88.9 45.72 90)
 			(hide yes)
@@
 			)
 		)
+		(pin "4"
+		)
+		(pin "3"
+		)
 		(pin "2"
 		)
 		(pin "1"
 		)
-		(pin "3"
-		)
-		(pin "4"
-		)
 		(instances

Commit message: DRC Error cleanups
Parts:
- R3, R5: footprint Resistor_SMD:R_0805_2012Metric_Pad1.20x1.40mm_HandSolder -> Resistor_SMD_JLC:R_0805_2012Metric_Pad1.20x1.40mm_HandSolder
Changed lines of the file:
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@@
 			)
 		)
-		(property "Footprint" "Resistor_SMD:R_0805_2012Metric_Pad1.20x1.40mm_HandSolder"
+		(property "Footprint" "Resistor_SMD_JLC:R_0805_2012Metric_Pad1.20x1.40mm_HandSolder"
 			(at 155.194 77.724 90)
 			(hide yes)
@@
 			)
 		)
-		(property "Footprint" "Resistor_SMD:R_0805_2012Metric_Pad1.20x1.40mm_HandSolder"
+		(property "Footprint" "Resistor_SMD_JLC:R_0805_2012Metric_Pad1.20x1.40mm_HandSolder"
 			(at 172.466 51.054 90)
 			(hide yes)

Commit message: DRC fixes
Parts:
- TP1, TP2, TP3: footprint TestPoint:TestPoint_Keystone_5005-5009_Compact -> TestPoint_JLC:TestPoint_Keystone_5005-5009_Compact_JLC
Changed lines of the file:
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@@
 			)
 		)
-		(property "Footprint" "TestPoint:TestPoint_Keystone_5005-5009_Compact"
+		(property "Footprint" "TestPoint_JLC:TestPoint_Keystone_5005-5009_Compact_JLC"
 			(at 157.48 34.29 0)
 			(hide yes)
@@
 			)
 		)
-		(property "Footprint" "TestPoint:TestPoint_Keystone_5005-5009_Compact"
+		(property "Footprint" "TestPoint_JLC:TestPoint_Keystone_5005-5009_Compact_JLC"
 			(at 186.69 64.77 0)
 			(hide yes)
@@
 			)
 		)
-		(property "Footprint" "TestPoint:TestPoint_Keystone_5005-5009_Compact"
+		(property "Footprint" "TestPoint_JLC:TestPoint_Keystone_5005-5009_Compact_JLC"
 			(at 167.64 40.64 0)
 			(hide yes)

Commit message: DRC cleanup
Parts:
- R10, R11, R6, R7, R8, R9: footprint Resistor_SMD:R_1206_3216Metric_Pad1.30x1.75mm_HandSolder -> Resistor_SMD_JLC:R_1206_3216Metric_Pad1.30x1.75mm_HandSolder
- R4: footprint Resistor_SMD:R_0805_2012Metric_Pad1.20x1.40mm_HandSolder -> Resistor_SMD_JLC:R_0805_2012Metric_Pad1.20x1.40mm_HandSolder
Changed lines of the file:
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@@
 			)
 		)
-		(property "Footprint" "Resistor_SMD:R_1206_3216Metric_Pad1.30x1.75mm_HandSolder"
+		(property "Footprint" "Resistor_SMD_JLC:R_1206_3216Metric_Pad1.30x1.75mm_HandSolder"
 			(at 230.886 66.294 90)
 			(hide yes)
@@
 			)
 		)
-		(property "Footprint" "Resistor_SMD:R_1206_3216Metric_Pad1.30x1.75mm_HandSolder"
+		(property "Footprint" "Resistor_SMD_JLC:R_1206_3216Metric_Pad1.30x1.75mm_HandSolder"
 			(at 180.086 52.324 90)
 			(hide yes)
@@
 			)
 		)
-		(property "Footprint" "Resistor_SMD:R_1206_3216Metric_Pad1.30x1.75mm_HandSolder"
+		(property "Footprint" "Resistor_SMD_JLC:R_1206_3216Metric_Pad1.30x1.75mm_HandSolder"
 			(at 194.056 38.354 90)
 			(hide yes)
@@
 			)
 		)
-		(property "Footprint" "Resistor_SMD:R_1206_3216Metric_Pad1.30x1.75mm_HandSolder"
+		(property "Footprint" "Resistor_SMD_JLC:R_1206_3216Metric_Pad1.30x1.75mm_HandSolder"
 			(at 190.246 65.024 90)
 			(hide yes)
@@
 			)
 		)
-		(property "Footprint" "Resistor_SMD:R_1206_3216Metric_Pad1.30x1.75mm_HandSolder"
+		(property "Footprint" "Resistor_SMD_JLC:R_1206_3216Metric_Pad1.30x1.75mm_HandSolder"
 			(at 230.886 51.054 90)
 			(hide yes)
@@
 			)
 		)
-		(property "Footprint" "Resistor_SMD:R_1206_3216Metric_Pad1.30x1.75mm_HandSolder"
+		(property "Footprint" "Resistor_SMD_JLC:R_1206_3216Metric_Pad1.30x1.75mm_HandSolder"
 			(at 197.866 68.834 90)
 			(hide yes)
@@
 			)
 		)
-		(property "Footprint" "Resistor_SMD:R_0805_2012Metric_Pad1.20x1.40mm_HandSolder"
+		(property "Footprint" "Resistor_SMD_JLC:R_0805_2012Metric_Pad1.20x1.40mm_HandSolder"
 			(at 158.496 47.244 90)
 			(hide yes)

Commit message: Rev 0.1.4 2026-07-16
Parts:
- J1: footprint TerminalBlock_Phoenix:PHOENIX_1731721 -> TerminalBlock_Phoenix_JLC:PHOENIX_1731721
Changed lines of the file:
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@@
 	(paper "A4")
 	(title_block
-		(date "2026-07-06")
-		(rev "0.1.3")
+		(date "2026-07-16")
+		(rev "0.1.4")
 	)
 	(text "~ 7mA"
@@
 			)
 		)
-		(property "Footprint" "TerminalBlock_Phoenix:PHOENIX_1731721"
+		(property "Footprint" "TerminalBlock_Phoenix_JLC:PHOENIX_1731721"
 			(at 24.13 55.88 0)
 			(hide yes)
