File: Dual15PowerSupply/Dual15PowerSupply.kicad_pcb (KiCad board)
At the start: 2 copper layers, 100 x 100 mm, 37 parts, among them J1 120VAC, J2 +/-15VDC, U1 LT3091, U2 LT3081

Commit message: in work
Parts:
- R5: footprint Resistor_SMD:R_1206_3216Metric_Pad1.30x1.75mm_HandSolder -> Resistor_SMD:R_0805_2012Metric_Pad1.20x1.40mm_HandSolder
- moved R8 6.71 mm to (168.0, 116.2), turned to 0 degrees
- moved R6 0.45 mm to (168.0, 111.5)
Routing:
- net Net-(U2-Imon): track 0.00 -> 4.02 mm
Changed lines of the file:
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@@
 		(embedded_fonts no)
 	)
-	(footprint "Resistor_SMD:R_1206_3216Metric_Pad1.30x1.75mm_HandSolder"
+	(footprint "Resistor_SMD:R_0805_2012Metric_Pad1.20x1.40mm_HandSolder"
 		(layer "F.Cu")
 		(at 176 120 -90)
-		(descr "Resistor SMD 1206 (3216 Metric), square (rectangular) end terminal, IPC-7351 nominal with elongated pad for handsoldering. (Body size source: IPC-SM-782 page 72, https://www.pcb-3d.com/wordpress/wp-content/uploads/ipc-sm-782a_amendment_1_and_2.pdf)")
+		(descr "Resistor SMD 0805 (2012 Metric), square (rectangular) end terminal, IPC-7351 nominal with elongated pad for handsoldering. (Body size source: IPC-SM-782 page 72, https://www.pcb-3d.com/wordpress/wp-content/uploads/ipc-sm-782a_amendment_1_and_2.pdf)")
 		(tags "resistor handsolder")
 		(property "Reference" "R5"
-			(at 3.5 0 90)
+			(at 0 -1.65 270)
 			(layer "F.SilkS")
 			(effects
@@
 		)
 		(property "Value" "4.99K"
-			(at 7 0 90)
+			(at 0 1.65 270)
 			(layer "F.Fab")
 			(effects
@@
 			)
 		)
-		(property "Datasheet" ""
-			(at 0 0 90)
+		(property "Datasheet" "https://www.mouser.com/datasheet/3/72/1/PYU_RT_1_TO_0_01_ROHS_L.pdf"
+			(at 0 0 270)
 			(layer "F.Fab")
 			(hide yes)
@@
 			)
 		)
-		(property "Description" "Resistor, US symbol"
-			(at 0 0 90)
+		(property "Description" "Resistor, 0805 4.99k.  1% 25ppm  (over spec'd but inexpensive part)"
+			(at 0 0 270)
 			(layer "F.Fab")
 			(hide yes)
@@
 		)
 		(property "KiLib_Generator" "SMD_2terminal_chip_molded"
-			(at 0 0 90)
+			(at 0 0 270)
 			(layer "F.SilkS")
 			(hide yes)
@@
 			)
 		)
-		(property "MPN" "RC1206FR-074K99L "
+		(property "MPN" "RT0805FRD074K99L"
 			(at 0 0 270)
 			(unlocked yes)
@@
 			)
 		)
-		(property "Mouser" "603-RC1206FR-074K99L "
+		(property "Mouser" "603-RT0805FRD074K99L "
 			(at 0 0 270)
 			(unlocked yes)
@@
 		(duplicate_pad_numbers_are_jumpers no)
 		(fp_line
-			(start -0.727064 0.91)
-			(end 0.727064 0.91)
+			(start -0.227064 0.735)
+			(end 0.227064 0.735)
 			(stroke
 				(width 0.12)
@@
 		)
 		(fp_line
-			(start -0.727064 -0.91)
-			(end 0.727064 -0.91)
+			(start -0.227064 -0.735)
+			(end 0.227064 -0.735)
 			(stroke
 				(width 0.12)
@@
 		)
 		(fp_rect
-			(start -2.45 -1.13)
-			(end 2.45 1.13)
+			(start -1.85 -0.95)
+			(end 1.85 0.95)
 			(stroke
 				(width 0.05)
@@
 		)
 		(fp_rect
-			(start -1.6 -0.8)
-			(end 1.6 0.8)
+			(start -1 -0.625)
+			(end 1 0.625)
 			(stroke
 				(width 0.1)
@@
 		)
 		(fp_text user "${REFERENCE}"
-			(at 0 0 90)
+			(at 0 0 270)
 			(layer "F.Fab")
 			(effects
 				(font
-					(size 0.8 0.8)
-					(thickness 0.12)
+					(size 0.5 0.5)
+					(thickness 0.08)
 				)
 			)
 		)
 		(pad "1" smd roundrect
-			(at -1.55 0 270)
-			(size 1.3 1.75)
+			(at -1 0 270)
+			(size 1.2 1.4)
 			(layers "F.Cu" "F.Mask" "F.Paste")
-			(roundrect_rratio 0.192308)
+			(roundrect_rratio 0.208333)
 			(net "Net-(U2-Imon)")
 			(pintype "passive")
 		)
 		(pad "2" smd roundrect
-			(at 1.55 0 270)
-			(size 1.3 1.75)
+			(at 1 0 270)
+			(size 1.2 1.4)
 			(layers "F.Cu" "F.Mask" "F.Paste")
-			(roundrect_rratio 0.192308)
+			(roundrect_rratio 0.208333)
 			(net "GND")
 			(pintype "passive")
 		)
 		(embedded_fonts no)
-		(model "${KICAD10_3DMODEL_DIR}/Resistor_SMD.3dshapes/R_1206_3216Metric.step"
+		(model "${KICAD10_3DMODEL_DIR}/Resistor_SMD.3dshapes/R_0805_2012Metric.step"
 			(offset
 				(xyz 0 0 0)
@@
 	(footprint "Resistor_SMD:R_1206_3216Metric_Pad1.30x1.75mm_HandSolder"
 		(layer "F.Cu")
-		(at 173.5 120 90)
+		(at 168 116.15)
 		(descr "Resistor SMD 1206 (3216 Metric), square (rectangular) end terminal, IPC-7351 nominal with elongated pad for handsoldering. (Body size source: IPC-SM-782 page 72, https://www.pcb-3d.com/wordpress/wp-content/uploads/ipc-sm-782a_amendment_1_and_2.pdf)")
 		(tags "resistor handsolder")
 		(property "Reference" "R8"
-			(at -3.5 0 90)
+			(at -3.5 0 0)
 			(layer "F.SilkS")
 			(effects
@@
 		)
 		(property "Value" "1.2k"
-			(at 0 -2 90)
+			(at 0.2 2.05 0)
 			(layer "F.Fab")
 			(effects
@@
 		)
 		(property "Datasheet" ""
-			(at 0 0 90)
+			(at 0 0 0)
 			(layer "F.Fab")
 			(hide yes)
@@
 		)
 		(property "Description" "Thin Film Resistor - 1206 1/4W 1.2K ohm 1% 50p pm"
-			(at 0 0 90)
+			(at 0 0 0)
 			(layer "F.Fab")
 			(hide yes)
@@
 		)
 		(property "KiLib_Generator" "SMD_2terminal_chip_molded"
-			(at 0 0 90)
+			(at 0 0 0)
 			(layer "F.SilkS")
 			(hide yes)
@@
 		)
 		(property "MPN" "RT1206FRE071K2L"
-			(at 0 0 90)
+			(at 0 0 0)
 			(unlocked yes)
 			(layer "F.Fab")
@@
 		)
 		(property "Mouser" "603-RT1206FRE071K2L "
-			(at 0 0 90)
+			(at 0 0 0)
 			(unlocked yes)
 			(layer "F.Fab")
@@
 		)
 		(fp_text user "${REFERENCE}"
-			(at 0 0 90)
+			(at 0 0 0)
 			(layer "F.Fab")
 			(effects
@@
 		)
 		(pad "1" smd roundrect
-			(at -1.55 0 90)
+			(at -1.55 0)
 			(size 1.3 1.75)
 			(layers "F.Cu" "F.Mask" "F.Paste")
@@
 		)
 		(pad "2" smd roundrect
-			(at 1.55 0 90)
+			(at 1.55 0)
 			(size 1.3 1.75)
 			(layers "F.Cu" "F.Mask" "F.Paste")
@@
 	(footprint "Resistor_SMD:R_1206_3216Metric_Pad1.30x1.75mm_HandSolder"
 		(layer "F.Cu")
-		(at 168.45 111.5 180)
+		(at 168 111.5 180)
 		(descr "Resistor SMD 1206 (3216 Metric), square (rectangular) end terminal, IPC-7351 nominal with elongated pad for handsoldering. (Body size source: IPC-SM-782 page 72, https://www.pcb-3d.com/wordpress/wp-content/uploads/ipc-sm-782a_amendment_1_and_2.pdf)")
 		(tags "resistor handsolder")
@@
 	)
 	(segment
+		(start 176.04 118.96)
+		(end 176 119)
+		(width 1)
+		(layer "F.Cu")
+		(net "Net-(U2-Imon)")
+	)
+	(segment
+		(start 176.04 115)
+		(end 176.04 118.96)
+		(width 1)
+		(layer "F.Cu")
+		(net "Net-(U2-Imon)")
+	)
+	(segment

Commit message: in progress
Parts:
- R3: footprint Resistor_SMD:R_1206_3216Metric_Pad1.30x1.75mm_HandSolder -> Resistor_SMD:R_0805_2012Metric_Pad1.20x1.40mm_HandSolder
- moved TP3 19.1 mm to (117.0, 104.0)
- moved C6 12.2 mm to (126.0, 125.0), turned to 90 degrees
- moved R11 11.2 mm to (132.0, 128.0)
- moved R3 10.8 mm to (122.0, 116.0), turned to 90 degrees
- moved U1 9.86 mm to (126.0, 115.0), turned to 0 degrees
- moved R7 8.06 mm to (122.0, 108.0)
- moved R9 7.07 mm to (131.0, 121.0), turned to 90 degrees
- moved TP2 7.07 mm to (175.0, 126.0)
- moved R8 4.14 mm to (171.0, 119.0)
- moved D4 2.27 mm to (139.0, 125.5), turned to 180 degrees
- moved C8 2.00 mm to (143.0, 112.0), turned to -90 degrees
- moved C5 0.57 mm to (169.6, 106.4)
- moved D3 0.50 mm to (163.0, 126.0)
- moved R10 0.50 mm to (167.5, 126.0)
- moved R6 0.20 mm to (168.0, 111.3)
Routing:
- net /+15VDC: track 0.00 -> 42.9 mm
- net Net-(U2-Imon): track 4.02 -> 12.6 mm
- net Net-(U2-TEMP): track 4.00 -> 9.25 mm
- net Net-(U2-SET): track 0.00 -> 5.22 mm
- net Net-(U2-Ilim): track 0.00 -> 4.39 mm
- net Net-(D3-K): track 0.00 -> 2.95 mm
- added copper zone on B.Cu, net /+15VDC
- added copper zone on F.Cu, net /+15VDC

Commit message: in wok
Parts:
- moved R7 7.50 mm to (127.2, 102.6)
- moved R3 2.00 mm to (122.0, 114.0), turned to -90 degrees
Routing:
- net /Vin-: track 11.4 -> 44.6 mm
- net Net-(U1-IMONN): track 0.00 -> 17.4 mm
- net Net-(U1-ILIM): track 0.00 -> 4.00 mm
Changed lines of the file:
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@@
 	(footprint "Resistor_SMD:R_0805_2012Metric_Pad1.20x1.40mm_HandSolder"
 		(layer "F.Cu")
-		(at 122 116 90)
+		(at 122 114 -90)
 		(descr "Resistor SMD 0805 (2012 Metric), square (rectangular) end terminal, IPC-7351 nominal with elongated pad for handsoldering. (Body size source: IPC-SM-782 page 72, https://www.pcb-3d.com/wordpress/wp-content/uploads/ipc-sm-782a_amendment_1_and_2.pdf)")
 		(tags "resistor handsolder")
@@
 		)
 		(property "MPN" "RC0805FR-0775KL "
-			(at 0 0 90)
+			(at 0 0 270)
 			(unlocked yes)
 			(layer "F.Fab")
@@
 		)
 		(property "Mouser" "603-RC0805FR-0775KL "
-			(at 0 0 90)
+			(at 0 0 270)
 			(unlocked yes)
 			(layer "F.Fab")
@@
 		(duplicate_pad_numbers_are_jumpers no)
 		(fp_line
-			(start -0.227064 -0.735)
-			(end 0.227064 -0.735)
+			(start -0.227064 0.735)
+			(end 0.227064 0.735)
 			(stroke
 				(width 0.12)
@@
 		)
 		(fp_line
-			(start -0.227064 0.735)
-			(end 0.227064 0.735)
+			(start -0.227064 -0.735)
+			(end 0.227064 -0.735)
 			(stroke
 				(width 0.12)
@@
 		)
 		(pad "1" smd roundrect
-			(at -1 0 90)
+			(at -1 0 270)
 			(size 1.2 1.4)
 			(layers "F.Cu" "F.Mask" "F.Paste")
@@
 		)
 		(pad "2" smd roundrect
-			(at 1 0 90)
+			(at 1 0 270)
 			(size 1.2 1.4)
 			(layers "F.Cu" "F.Mask" "F.Paste")
@@
 	(footprint "Resistor_SMD:R_1206_3216Metric_Pad1.30x1.75mm_HandSolder"
 		(layer "F.Cu")
-		(at 122 108 -90)
+		(at 127.2 102.6 -90)
 		(descr "Resistor SMD 1206 (3216 Metric), square (rectangular) end terminal, IPC-7351 nominal with elongated pad for handsoldering. (Body size source: IPC-SM-782 page 72, https://www.pcb-3d.com/wordpress/wp-content/uploads/ipc-sm-782a_amendment_1_and_2.pdf)")
 		(tags "resistor handsolder")
@@
 	)
 	(segment
+		(start 114 115)
+		(end 116 113)
+		(width 1)
+		(layer "F.Cu")
+		(net "/Vin-")
+	)
+	(segment
+		(start 116 113)
+		(end 122 113)
+		(width 1)
+		(layer "F.Cu")
+		(net "/Vin-")
+	)
+	(segment
+		(start 128.582792 108.8)
+		(end 129.81 110.027208)
+		(width 1.5)
+		(layer "B.Cu")
+		(net "/Vin-")
+	)
+	(segment
+		(start 120.2 108.8)
+		(end 128.582792 108.8)
+		(width 1.5)
+		(layer "B.Cu")
+		(net "/Vin-")
+	)
+	(segment
+		(start 129.81 110.027208)
+		(end 129.81 111.3)
+		(width 1.5)
+		(layer "B.Cu")
+		(net "/Vin-")
+	)
+	(segment
 		(start 109 105.66)
 		(end 114 110.66)
@@
 	)
 	(segment
+		(start 114 115)
+		(end 120.2 108.8)
+		(width 1.5)
+		(layer "B.Cu")
+		(net "/Vin-")
+	)
+	(segment
+		(start 128.54 112.57)
+		(end 129.81 111.3)
+		(width 1)
+		(layer "B.Cu")
+		(net "/Vin-")
+	)
+	(segment
+		(start 128.54 115)
+		(end 128.54 112.57)
+		(width 1)
+		(layer "B.Cu")
+		(net "/Vin-")
+	)
+	(segment
 		(start 176.04 118.96)
 		(end 176 119)
@@
 	)
 	(segment
+		(start 122 115)
+		(end 126 115)
+		(width 1)
+		(layer "F.Cu")
+		(net "Net-(U1-ILIM)")
+	)
+	(segment
 		(start 131.19 37.3)
 		(end 143.8 37.3)
@@
 		(net "Net-(U2-SET)")
 	)
+	(segment
+		(start 117 104)
+		(end 117.2 104)
+		(width 1)
+		(layer "F.Cu")
+		(net "Net-(U1-IMONN)")
+	)
+	(segment
+		(start 117.2 104)
+		(end 117.35 104.15)
+		(width 1)
+		(layer "F.Cu")
+		(net "Net-(U1-IMONN)")
+	)
+	(segment
+		(start 127.27 111.3)
+		(end 127.27 104.22)
+		(width 1)
+		(layer "F.Cu")
+		(net "Net-(U1-IMONN)")
+	)
+	(segment
+		(start 117.35 104.15)
+		(end 127.2 104.15)
+		(width 1)
+		(layer "F.Cu")
+		(net "Net-(U1-IMONN)")
+	)
+	(segment
+		(start 127.27 104.22)
+		(end 127.2 104.15)
+		(width 1)
+		(layer "F.Cu")
+		(net "Net-(U1-IMONN)")
+	)
 	(zone
 		(net "/+15VDC")
@@
 		)
 		(min_thickness 0.3)
-		(fill
+		(fill yes
 			(thermal_gap 0.5)
 			(thermal_bridge_width 0.5)
